Commit message: Don't use surface adjustments

File: orca_gazebo/urdf/orca.urdf.xacro (robot description, xacro)
@@ -24,5 +24,5 @@
   <xacro:property name="REVERSE_FORCE" value="40"/>
   <xacro:property name="HAS_TETHER" default="false"/>
-  <xacro:property name="SURFACE" default="10"/>
+  <xacro:property name="SURFACE" default="0"/>
   <!-- Physics properties -->
   <xacro:property name="FLUID_DENSITY" value="1029"/>
@@ -225,4 +225,5 @@
         <ros_topic>/barometer</ros_topic>
         <fluid_density>${FLUID_DENSITY}</fluid_density>
+        <surface>${SURFACE}</surface>
       </plugin>
     </sensor>

Commit message: Start on new map-driven missions, and new controller

File: orca_gazebo/urdf/orca.urdf.xacro (robot description, xacro)
@@ -236,16 +236,4 @@
   </gazebo>
   <!--
-    The OrcaGPSPlugin simulates a GPS receiver attached to an ROV.
-    When it goes underwater, the GPS signal is lost.
-  -->
-  <gazebo>
-    <plugin name="OrcaGPSPlugin" filename="libOrcaGPSPlugin.so">
-      <link name="base_link">
-        <ros_topic>/gps</ros_topic>
-        <mast_height>1</mast_height>
-      </link>
-    </plugin>
-  </gazebo>
-  <!--
     The OrcaGroundTruthPlugin publishes a ground truth pose.
   -->
