Commit message: Use /clock if available

File: orca_gazebo/urdf/orca.urdf (robot description, URDF)
Before this commit: robot orca, 8 links, 7 joints
Joints:
- joint camera_joint: origin xyz=0 0 -0.2 rpy=0 0 0 -> xyz=0 0 -0.2 rpy=0 1.57079 0

Commit message: Updated config to more closely match the upcoming pool tests

File: orca_gazebo/urdf/orca.urdf (robot description, URDF)
Before this commit: robot orca, 8 links, 7 joints
Links:
- removed link camera_link
- added link left_camera_link; visual sphere radius=0.026
- added link right_camera_link; visual sphere radius=0.026
- link base_link: geometry collision box size=0.457 0.338 0.254; visual box size=0.15 0.09 0.08
Joints:
- removed joint camera_joint
- added joint left_camera_joint: type fixed, parent base_link, child left_camera_link, origin xyz=-0.15 0.18 -0.0675 rpy=0 1.57079 0, axis 0 1 0
- added joint right_camera_joint: type fixed, parent base_link, child right_camera_link, origin xyz=-0.15 -0.18 -0.0675 rpy=0 1.57079 0, axis 0 1 0

File: orca_gazebo/urdf/orca.urdf.xacro (robot description, xacro)
@@ -1,5 +1,7 @@
 <?xml version="1.0"?>
-<!-- Coordinates are: x forward, y left, z up; rotation is: roll right, pitch forward, yaw left -->
-<!-- See http://www.ros.org/reps/rep-0103.html for details -->
+<!--
+  Coordinates are: x forward, y left, z up; rotation is: roll right, pitch forward, yaw left.
+  See http://www.ros.org/reps/rep-0103.html for details.
+-->
 <robot name="orca" xmlns:xacro="http://ros.org/wiki/xacro">
   <!-- Orca constants -->
@@ -33,4 +35,5 @@
   <material name="gray"><color rgba="0.5 0.5 0.5 1.0"/></material>
   <material name="blue"><color rgba="0.5 0.5 1.0 1.0"/></material>
+  <material name="red"><color rgba="1.0 0.0 0.0 1.0"/></material>
   <!-- Thruster origins -->
   <xacro:property name="front_right_origin">
@@ -55,23 +58,24 @@
   <xacro:macro name="t200" params="name *origin">
     <link name="t200_link_${name}">
+      <!-- Front cone -->
       <visual>
         <origin xyz="0 0 0"/>
         <geometry><sphere radius="0.02"/></geometry>
-        <material name="gray"/>
+        <material name="gray"/> <!-- All visual elements in this link pick up this material -->
       </visual>
+      <!-- Rear cone -->
       <visual>
         <origin xyz="0 0 -0.07"/>
         <geometry><sphere radius="0.02"/></geometry>
-        <material name="gray"/>
       </visual>
+      <!-- Thruster body -->
       <visual>
         <origin xyz="0 0 -0.035"/>
         <geometry><cylinder length="0.07" radius="0.02"/></geometry>
-        <material name="gray"/>
       </visual>
+      <!-- Propeller guard -->
       <visual>
         <origin xyz="0 0 -0.0225"/>
         <geometry><cylinder length="0.045" radius="0.045"/></geometry>
-        <material name="gray"/>
       </visual>
     </link>
@@ -84,4 +88,5 @@
   <!-- Base link -->
   <link name="base_link">
+    <!-- Inertial -->
     <inertial>
       <origin xyz="0 0 ${MASS_Z}"/> <!-- Center of mass -->
@@ -89,4 +94,5 @@
       <inertia ixx="${IXX}" ixy="0.0" ixz="0.0" iyy="${IYY}" iyz="0.0" izz="${IZZ}"/>
     </inertial>
+    <!-- Float -->
     <visual>
       <origin xyz="${FLOAT_X} ${FLOAT_Y} ${FLOAT_Z}"/>
@@ -94,38 +100,81 @@
       <material name="blue"/>
     </visual>
+    <!-- Float -->
     <visual>
       <origin xyz="${FLOAT_X} ${-FLOAT_Y} ${FLOAT_Z}"/>
       <geometry><box size="0.15 0.09 0.08"/></geometry>
-      <material name="blue"/>
-    </visual>
+    </visual>
+    <!-- Float -->
     <visual>
       <origin xyz="${-FLOAT_X} ${FLOAT_Y} ${FLOAT_Z}"/>
       <geometry><box size="0.15 0.09 0.08"/></geometry>
-      <material name="blue"/>
-    </visual>
+    </visual>
+    <!-- Float -->
     <visual>
       <origin xyz="${-FLOAT_X} ${-FLOAT_Y} ${FLOAT_Z}"/>
       <geometry><box size="0.15 0.09 0.08"/></geometry>
-      <material name="blue"/>
-    </visual>
+    </visual>
+    <!-- Electronics tube -->
     <visual>
       <origin xyz="0 0 0.063" rpy="0 ${PI/2} 0"/>
       <geometry><cylinder length="0.32" radius="0.055"/></geometry>
-      <material name="blue"/>
-    </visual>
+    </visual>
+    <!-- Front-facing camera hemisphere -->
     <visual>
       <origin xyz="0.16 0 0.063" rpy="0 ${PI/2} 0"/>
       <geometry><sphere radius="0.052"/></geometry>
-      <material name="blue"/>
-    </visual>
+    </visual>
+    <!-- Battery tube -->
     <visual>
       <origin xyz="0 0 -0.05" rpy="0 ${PI/2} 0"/>
       <geometry><cylinder length="0.25" radius="0.045"/></geometry>
-      <material name="blue"/>
-    </visual>
+    </visual>
+    <!-- Left down-facing camera tube -->
+    <visual>
+      <origin xyz="-0.15 0.18 0" rpy="0 0 0"/>
+      <geometry><cylinder length="0.135" radius="0.0275"/></geometry>
+    </visual>
+    <!-- Right down-facing camera tube -->
+    <visual>
+      <origin xyz="-0.15 -0.18 0" rpy="0 0 0"/>
+      <geometry><cylinder length="0.135" radius="0.0275"/></geometry>
+    </visual>
+    <!-- Collision region -->
     <collision>
       <geometry><box size="${LENGTH} ${WIDTH} ${HEIGHT}"/></geometry>
     </collision>
   </link>
+  <!-- Left down-facing camera -->
+  <link name="left_camera_link">
+    <!-- Camera hemisphere -->
+    <visual>
+      <origin xyz="0 0 0" rpy="0 0 0"/>
+      <geometry><sphere radius="0.026"/></geometry>
+      <material name="red"/>
+    </visual>
+  </link>
+  <!-- Attach left down-facing camera to base_link -->
+  <joint name="left_camera_joint" type="fixed">
+    <axis xyz="0 1 0" />
+    <origin xyz="-0.15 0.18 -0.0675" rpy="0 1.57079 0"/>
+    <parent link="base_link"/>
+    <child link="left_camera_link"/>
+  </joint>
+  <!-- Right down-facing camera -->
+  <link name="right_camera_link">
+    <!-- Camera hemisphere -->
+    <visual>
+      <origin xyz="0 0 0" rpy="0 0 0"/>
+      <geometry><sphere radius="0.026"/></geometry>
+      <material name="red"/>
+    </visual>
+  </link>
+  <!-- Attach right down-facing camera to base_link -->
+  <joint name="right_camera_joint" type="fixed">
+    <axis xyz="0 1 0" />
+    <origin xyz="-0.15 -0.18 -0.0675" rpy="0 1.57079 0"/>
+    <parent link="base_link"/>
+    <child link="right_camera_link"/>
+  </joint>
   <!-- Attach thrusters to the base_link -->
   <xacro:t200 name="front_right">
@@ -176,5 +225,5 @@
   <!--
     The OrcaThrusterPlugin turns ROS messages into thrust forces. Each message contains an array of thrust efforts [-1.0, 1.0].
-    The URDF to SDF translation nukes the joints, so we need to copy/paste the joint locations here.
+    The URDF to SDF translation nukes the joints, so joint locations must appear here.
   -->
   <gazebo>
@@ -244,3 +293,46 @@
     </plugin>
   </gazebo>
+  <!--
+    The camera_controller plugin (wraps a Gazebo camera sensor) simulates a camera driver.
+    Left down-facing camera driver:
+  -->
+  <gazebo reference="left_camera_link">
+    <sensor type="camera" name="left_camera">
+      <update_rate>30.0</update_rate>
+      <camera name="head">
+        <horizontal_fov>1.92</horizontal_fov>
+        <image>
+          <width>800</width>
+          <height>600</height>
+          <format>R8G8B8</format>
+        </image>
+        <clip>
+          <near>0.02</near>
+          <far>300</far>
+        </clip>
+        <noise>
+          <type>gaussian</type>
+          <!-- Noise is sampled independently per pixel on each frame.
+               That pixel's noise value is added to each of its color
+               channels, which at that point lie in the range [0,1]. -->
+          <mean>0.0</mean>
+          <stddev>0.007</stddev>
+        </noise>
+      </camera>
+      <plugin name="camera_controller" filename="libgazebo_ros_camera.so">
+        <alwaysOn>true</alwaysOn>
+        <updateRate>0.0</updateRate>
+        <cameraName>orca/left_camera</cameraName>
+        <imageTopicName>image_raw</imageTopicName>
+        <cameraInfoTopicName>camera_info</cameraInfoTopicName>
+        <frameName>left_camera_link</frameName>
+        <hackBaseline>0.07</hackBaseline>
+        <distortionK1>0.0</distortionK1>
+        <distortionK2>0.0</distortionK2>
+        <distortionK3>0.0</distortionK3>
+        <distortionT1>0.0</distortionT1>
+        <distortionT2>0.0</distortionT2>
+      </plugin>
+    </sensor>
+  </gazebo>
 </robot>
