Commit message: Create pt2, hardware build for pool test 2

File: orca_description/urdf/pt2.urdf (robot description, URDF)
Before this commit: robot orca, 9 links, 8 joints
Links:
- removed link left_camera_link
- removed link right_camera_link
- added link forward_camera_link; visual sphere radius=0.052
- link base_link: geometry collision box size=0.457 0.338 0.254; visual box size=0.15 0.09 0.08
Joints:
- removed joint left_camera_joint
- removed joint right_camera_joint
- added joint forward_camera_joint: type fixed, parent base_link, child forward_camera_link, origin xyz=0.16 0 0.063 rpy=0 0 0, axis 0 1 0

File: orca_description/urdf/pt2.urdf.xacro (robot description, xacro)
@@ -1,5 +1,5 @@
 <?xml version="1.0"?>
 <!--
-  Generic version of Orca
+  Hardware build for pool test #2
 -->
 <robot name="orca" xmlns:xacro="http://ros.org/wiki/xacro">
@@ -119,23 +119,8 @@
       <geometry><cylinder length="0.32" radius="0.055"/></geometry>
     </visual>
-    <!-- Front-facing camera hemisphere -->
-    <visual>
-      <origin xyz="0.16 0 0.063" rpy="0 ${PI/2} 0"/>
-      <geometry><sphere radius="0.052"/></geometry>
-    </visual>
     <!-- Battery tube -->
     <visual>
       <origin xyz="0 0 -0.05" rpy="0 ${PI/2} 0"/>
       <geometry><cylinder length="0.25" radius="0.045"/></geometry>
-    </visual>
-    <!-- Left down-facing camera tube -->
-    <visual>
-      <origin xyz="-0.15 0.18 0" rpy="0 0 0"/>
-      <geometry><cylinder length="0.135" radius="0.0275"/></geometry>
-    </visual>
-    <!-- Right down-facing camera tube -->
-    <visual>
-      <origin xyz="-0.15 -0.18 0" rpy="0 0 0"/>
-      <geometry><cylinder length="0.135" radius="0.0275"/></geometry>
     </visual>
     <!-- Collision region -->
@@ -144,35 +129,19 @@
     </collision>
   </link>
-  <!-- Left down-facing camera -->
-  <link name="left_camera_link">
+  <!-- Forward camera -->
+  <link name="forward_camera_link">
     <!-- Camera hemisphere -->
     <visual>
       <origin xyz="0 0 0" rpy="0 0 0"/>
-      <geometry><sphere radius="0.026"/></geometry>
+      <geometry><sphere radius="0.052"/></geometry>
       <material name="red"/>
     </visual>
   </link>
-  <!-- Attach left down-facing camera to base_link -->
-  <joint name="left_camera_joint" type="fixed">
+  <!-- Attach forward camera to base_link -->
+  <joint name="forward_camera_joint" type="fixed">
     <axis xyz="0 1 0" />
-    <origin xyz="-0.15 0.18 -0.0675" rpy="0 ${PI/2} 0"/>
+    <origin xyz="0.16 0 0.063" rpy="0 0 0"/>
     <parent link="base_link"/>
-    <child link="left_camera_link"/>
-  </joint>
-  <!-- Right down-facing camera -->
-  <link name="right_camera_link">
-    <!-- Camera hemisphere -->
-    <visual>
-      <origin xyz="0 0 0" rpy="0 0 0"/>
-      <geometry><sphere radius="0.026"/></geometry>
-      <material name="red"/>
-    </visual>
-  </link>
-  <!-- Attach right down-facing camera to base_link -->
-  <joint name="right_camera_joint" type="fixed">
-    <axis xyz="0 1 0" />
-    <origin xyz="-0.15 -0.18 -0.0675" rpy="0 1.57079 0"/>
-    <parent link="base_link"/>
-    <child link="right_camera_link"/>
+    <child link="forward_camera_link"/>
   </joint>
   <!-- Attach thrusters to the base_link -->
@@ -273,29 +242,9 @@
   </gazebo>
   <!--
-    The OrcaIMUPlugin (wraps a Gazebo IMU sensor) simulates an IMU sensor such as the Phidgets 1044.
-  -->
-  <gazebo reference="base_link">
-    <gravity>true</gravity>
-    <sensor name="imu_sensor" type="imu">
-      <update_rate>50</update_rate> <!-- Gazebeo max seems to be 50Hz -->
-      <plugin name="OrcaIMUPlugin" filename="libOrcaIMUPlugin.so" />
-      <pose>0 0 0 0 0 0</pose>
-    </sensor>
-  </gazebo>
-  <!--
-    The OrcaGroundTruthPlugin publishes a ground truth pose.
-  -->
-  <gazebo>
-    <plugin name="OrcaGroundTruthPlugin" filename="libOrcaGroundTruthPlugin.so">
-      <link name="base_link" />
-      <ros_topic>/ground_truth</ros_topic>
-    </plugin>
-  </gazebo>
-  <!--
     The camera_controller plugin (wraps a Gazebo camera sensor) simulates a camera driver.
-    Left down-facing camera driver:
-  -->
-  <gazebo reference="left_camera_link">
-    <sensor type="camera" name="left_camera">
+    Forward-facing camera driver:
+  -->
+  <gazebo reference="forward_camera_link">
+    <sensor type="camera" name="forward_camera">
       <update_rate>30.0</update_rate>
       <camera name="head">
@@ -322,8 +271,8 @@
         <alwaysOn>true</alwaysOn>
         <updateRate>0.0</updateRate>
-        <cameraName>orca/left_camera</cameraName>
+        <cameraName>orca/forward_camera</cameraName>
         <imageTopicName>image_raw</imageTopicName>
         <cameraInfoTopicName>camera_info</cameraInfoTopicName>
-        <frameName>left_camera_link</frameName>
+        <frameName>forward_camera_link</frameName>
         <hackBaseline>0.07</hackBaseline>
         <distortionK1>0.0</distortionK1>

Commit message: Add forward_camera_frame, add record.bash

File: orca_description/urdf/pt2.urdf (robot description, URDF)
Before this commit: robot orca, 8 links, 7 joints
Links:
- added link forward_camera_frame
Joints:
- removed joint forward_camera_joint
- added joint forward_camera_frame_joint: type fixed, parent forward_camera_link, child forward_camera_frame, origin xyz=0 0 0 rpy=-1.57079632679 0 -1.57079632679
- added joint forward_camera_link_joint: type fixed, parent base_link, child forward_camera_link, origin xyz=0.16 0 0.063 rpy=0 0 0

File: orca_description/urdf/pt2.urdf.xacro (robot description, xacro)
@@ -129,5 +129,5 @@
     </collision>
   </link>
-  <!-- Forward camera -->
+  <!-- Forward camera link -->
   <link name="forward_camera_link">
     <!-- Camera hemisphere -->
@@ -138,10 +138,17 @@
     </visual>
   </link>
-  <!-- Attach forward camera to base_link -->
-  <joint name="forward_camera_joint" type="fixed">
-    <axis xyz="0 1 0" />
+  <!-- Attach forward_camera_link to base_link -->
+  <joint name="forward_camera_link_joint" type="fixed">
     <origin xyz="0.16 0 0.063" rpy="0 0 0"/>
     <parent link="base_link"/>
     <child link="forward_camera_link"/>
+  </joint>
+  <!-- Forward camera frame -->
+  <link name="forward_camera_frame"/>
+  <!-- Attach forward_camera_frame to forward_camera_link -->
+  <joint name="forward_camera_frame_joint" type="fixed">
+    <origin xyz="0 0 0" rpy="${-PI/2} 0 ${-PI/2}"/>
+    <parent link="forward_camera_link"/>
+    <child link="forward_camera_frame"/>
   </joint>
   <!-- Attach thrusters to the base_link -->

Commit message: Practice PID tuning

File: orca_description/urdf/pt2.urdf (robot description, URDF)
Before this commit: robot orca, 9 links, 8 joints
Links:
- removed link forward_camera_frame
Joints:
- removed joint forward_camera_frame_joint

File: orca_description/urdf/pt2.urdf.xacro (robot description, xacro)
@@ -144,12 +144,12 @@
     <child link="forward_camera_link"/>
   </joint>
-  <!-- Forward camera frame -->
-  <link name="forward_camera_frame"/>
-  <!-- Attach forward_camera_frame to forward_camera_link -->
-  <joint name="forward_camera_frame_joint" type="fixed">
-    <origin xyz="0 0 0" rpy="${-PI/2} 0 ${-PI/2}"/>
-    <parent link="forward_camera_link"/>
-    <child link="forward_camera_frame"/>
-  </joint>
+<!--  &lt;!&ndash; Forward camera frame &ndash;&gt;-->
+<!--  <link name="forward_camera_frame"/>-->
+<!--  &lt;!&ndash; Attach forward_camera_frame to forward_camera_link &ndash;&gt;-->
+<!--  <joint name="forward_camera_frame_joint" type="fixed">-->
+<!--    <origin xyz="0 0 0" rpy="${-PI/2} 0 ${-PI/2}"/>-->
+<!--    <parent link="forward_camera_link"/>-->
+<!--    <child link="forward_camera_frame"/>-->
+<!--  </joint>-->
   <!-- Attach thrusters to the base_link -->
   <xacro:t200 name="front_right">
