Commit message: Fuse fiducial_vlam and barometer sensors into a single pose, remove ground_truth plugin, other cleanups

File: orca_description/urdf/orca.urdf.xacro (robot description, xacro)
@@ -266,5 +266,5 @@
   <gazebo reference="base_link">
     <sensor name="barometer_sensor" type="altimeter">
-      <update_rate>50</update_rate> <!-- Match orca_driver rate -->
+      <update_rate>10</update_rate> <!-- Match orca_driver rate -->
       <plugin name="OrcaBarometerPlugin" filename="libOrcaBarometerPlugin.so">
         <fluid_density>${FLUID_DENSITY}</fluid_density>
@@ -282,13 +282,4 @@
       <pose>0 0 0 0 0 0</pose>
     </sensor>
-  </gazebo>
-  <!--
-    The OrcaGroundTruthPlugin publishes a ground truth pose.
-  -->
-  <gazebo>
-    <plugin name="OrcaGroundTruthPlugin" filename="libOrcaGroundTruthPlugin.so">
-      <link name="base_link" />
-      <ros_topic>/ground_truth</ros_topic>
-    </plugin>
   </gazebo>
   <!--

File: orca_description/urdf/pt2.urdf.xacro (robot description, xacro)
@@ -242,5 +242,5 @@
   <gazebo reference="base_link">
     <sensor name="barometer_sensor" type="altimeter">
-      <update_rate>50</update_rate> <!-- Match orca_driver rate -->
+      <update_rate>10</update_rate> <!-- Match orca_driver rate -->
       <plugin name="OrcaBarometerPlugin" filename="libOrcaBarometerPlugin.so">
         <fluid_density>${FLUID_DENSITY}</fluid_density>

Commit message: Split base_node and filter_node; add messages queues to filter

File: orca_description/urdf/orca.urdf.xacro (robot description, xacro)
@@ -27,5 +27,5 @@
   <xacro:property name="SURFACE" default="0"/>
   <!-- Physics properties -->
-  <xacro:property name="FLUID_DENSITY" value="1029"/>
+  <xacro:property name="FLUID_DENSITY" value="997"/>
   <xacro:property name="DISPLACED_MASS" value="${TOTAL_VOLUME*FLUID_DENSITY}"/>
   <!-- General constants -->

File: orca_description/urdf/pt2.urdf.xacro (robot description, xacro)
@@ -27,5 +27,5 @@
   <xacro:property name="SURFACE" default="0"/>
   <!-- Physics properties -->
-  <xacro:property name="FLUID_DENSITY" value="1029"/>
+  <xacro:property name="FLUID_DENSITY" value="997"/>
   <xacro:property name="DISPLACED_MASS" value="${TOTAL_VOLUME*FLUID_DENSITY}"/>
   <!-- General constants -->
