Commit message: Tried to add a camera, but gazebo_ros_pkgs doesn't support this yet

File: orca_description/urdf/orca.urdf (robot description, URDF)
Before this commit: robot orca, 7 links, 6 joints
Links:
- added link camera_link, mass 1e-5; collision box size=0.05 0.05 0.05; visual box size=0.05 0.05 0.05
Joints:
- added joint camera_joint: type fixed, parent base_link, child camera_link, origin xyz=0 0 -0.2 rpy=0 0 0, axis 0 1 0

File: orca_description/urdf/orca.urdf.xacro (robot description, xacro)
@@ -257,5 +257,5 @@
     <plugin name="OrcaGroundTruthPlugin" filename="libOrcaGroundTruthPlugin.so">
       <link name="base_link" />
-      <ros_topic>/gps</ros_topic>
+      <ros_topic>/ground_truth</ros_topic>
       <surface>${SURFACE}</surface>
     </plugin>

Commit message: Multiple cameras, parse URDF, filter pose not odom, ROV hold pressure not z

File: orca_description/urdf/orca.urdf (robot description, URDF)
Before this commit: robot orca, 9 links, 8 joints
Links:
- added link baro_link; visual cylinder length=0.01 radius=0.01
- added link forward_camera_frame
- added link forward_camera_link; visual sphere radius=0.052
- added link left_camera_frame
- added link right_camera_frame
- link base_link: mass 10 -> 9.75; geometry collision box size=0.457 0.338 0.254; visual box size=0.15 0.09 0.08
Joints:
- added joint baro_joint: type fixed, parent base_link, child baro_link, origin xyz=-0.16 0 0 rpy=0 0 0
- added joint forward_camera_frame_joint: type fixed, parent base_link, child forward_camera_frame, origin xyz=0.16 0 0.063 rpy=-1.57079632679 0 -1.57079632679
- added joint forward_camera_joint: type fixed, parent base_link, child forward_camera_link, origin xyz=0.16 0 0.063 rpy=0 0 0
- added joint left_camera_frame_joint: type fixed, parent base_link, child left_camera_frame, origin xyz=-0.15 0.18 -0.0675 rpy=3.14159265359 0 -1.57079632679
- added joint right_camera_frame_joint: type fixed, parent base_link, child right_camera_frame, origin xyz=-0.15 -0.18 -0.0675 rpy=3.14159265359 0 -1.57079632679

File: orca_description/urdf/orca.urdf.xacro (robot description, xacro)
@@ -1,328 +1,420 @@
 <?xml version="1.0"?>
-<!--
-  Generic version of Orca
--->
 <robot name="orca" xmlns:xacro="http://ros.org/wiki/xacro">
-  <!-- Orca constants -->
-  <xacro:property name="TOTAL_MASS" value="10"/>
-  <xacro:property name="TOTAL_VOLUME" value="0.01"/>
-  <xacro:property name="LENGTH" value="0.457"/>
-  <xacro:property name="WIDTH" value="0.338"/>
-  <xacro:property name="HEIGHT" value="0.254"/>
-  <xacro:property name="IXX" value="${TOTAL_MASS / 12 * (WIDTH * WIDTH + HEIGHT * HEIGHT)}"/>
-  <xacro:property name="IYY" value="${TOTAL_MASS / 12 * (LENGTH * LENGTH + HEIGHT * HEIGHT)}"/>
-  <xacro:property name="IZZ" value="${TOTAL_MASS / 12 * (LENGTH * LENGTH + WIDTH * WIDTH)}"/>
-  <xacro:property name="FLOAT_X" value="0.12"/>
-  <xacro:property name="FLOAT_Y" value="0.11"/>
-  <xacro:property name="FLOAT_Z" value="0.07"/>
-  <xacro:property name="THRUSTER_X" value="0.15"/>
-  <xacro:property name="THRUSTER_Y" value="0.09"/>
-  <xacro:property name="THRUSTER_Z" value="-0.009"/>
-  <xacro:property name="VERT_THRUSTER_Y" value="0.105"/>
-  <xacro:property name="VERT_THRUSTER_Z" value="0.09"/>
-  <xacro:property name="MASS_Z" value="0.011"/>
-  <xacro:property name="FORWARD_FORCE" value="50"/>
-  <xacro:property name="REVERSE_FORCE" value="40"/>
-  <xacro:property name="HAS_TETHER" default="false"/>
-  <xacro:property name="SURFACE" default="0"/>
-  <!-- Physics properties -->
-  <xacro:property name="FLUID_DENSITY" value="997"/>
-  <xacro:property name="DISPLACED_MASS" value="${TOTAL_VOLUME*FLUID_DENSITY}"/>
-  <!-- General constants -->
-  <xacro:property name="PI" value="3.1415926535897931"/>
-  <!-- Materials -->
-  <material name="gray"><color rgba="0.5 0.5 0.5 1.0"/></material>
-  <material name="blue"><color rgba="0.5 0.5 1.0 1.0"/></material>
-  <material name="red"><color rgba="1.0 0.0 0.0 1.0"/></material>
-  <!-- Thruster origins -->
-  <xacro:property name="front_right_origin">
-    <origin xyz="${THRUSTER_X} ${-THRUSTER_Y} ${THRUSTER_Z}" rpy="0 ${PI/2} ${PI/4}"/>
-  </xacro:property>
-  <xacro:property name="front_left_origin">
-    <origin xyz="${THRUSTER_X} ${THRUSTER_Y} ${THRUSTER_Z}" rpy="0 ${PI/2} ${-PI/4}"/>
-  </xacro:property>
-  <xacro:property name="rear_right_origin">
-    <origin xyz="${-THRUSTER_X} ${-THRUSTER_Y} ${THRUSTER_Z}" rpy="0 ${PI/2} ${PI*3/4}"/>
-  </xacro:property>
-  <xacro:property name="rear_left_origin">
-    <origin xyz="${-THRUSTER_X} ${THRUSTER_Y} ${THRUSTER_Z}" rpy="0 ${PI/2} ${-PI*3/4}"/>
-  </xacro:property>
-  <xacro:property name="vertical_right_origin">
-    <origin xyz="0 ${-VERT_THRUSTER_Y} ${VERT_THRUSTER_Z}" rpy="0 0 0"/>
-  </xacro:property>
-  <xacro:property name="vertical_left_origin">
-    <origin xyz="0 ${VERT_THRUSTER_Y} ${VERT_THRUSTER_Z}" rpy="0 0 0"/>
-  </xacro:property>
-  <!-- Thruster macro -->
-  <xacro:macro name="t200" params="name *origin">
-    <link name="t200_link_${name}">
-      <!-- Front cone -->
-      <visual>
-        <origin xyz="0 0 0"/>
-        <geometry><sphere radius="0.02"/></geometry>
-        <material name="gray"/> <!-- All visual elements in this link pick up this material -->
-      </visual>
-      <!-- Rear cone -->
-      <visual>
-        <origin xyz="0 0 -0.07"/>
-        <geometry><sphere radius="0.02"/></geometry>
-      </visual>
-      <!-- Thruster body -->
-      <visual>
-        <origin xyz="0 0 -0.035"/>
-        <geometry><cylinder length="0.07" radius="0.02"/></geometry>
-      </visual>
-      <!-- Propeller guard -->
-      <visual>
-        <origin xyz="0 0 -0.0225"/>
-        <geometry><cylinder length="0.045" radius="0.045"/></geometry>
-      </visual>
+    <!-- Orca constants -->
+    <xacro:property name="TOTAL_MASS" value="9.75"/>  <!-- 9.75 floats in freshwater, 10.0 for seawater -->
+    <xacro:property name="TOTAL_VOLUME" value="0.01"/>
+    <xacro:property name="LENGTH" value="0.457"/>
+    <xacro:property name="WIDTH" value="0.338"/>
+    <xacro:property name="HEIGHT" value="0.254"/>
+    <xacro:property name="IXX" value="${TOTAL_MASS / 12 * (WIDTH * WIDTH + HEIGHT * HEIGHT)}"/>
+    <xacro:property name="IYY" value="${TOTAL_MASS / 12 * (LENGTH * LENGTH + HEIGHT * HEIGHT)}"/>
+    <xacro:property name="IZZ" value="${TOTAL_MASS / 12 * (LENGTH * LENGTH + WIDTH * WIDTH)}"/>
+    <xacro:property name="FLOAT_X" value="0.12"/>
+    <xacro:property name="FLOAT_Y" value="0.11"/>
+    <xacro:property name="FLOAT_Z" value="0.07"/>
+    <xacro:property name="THRUSTER_X" value="0.15"/>
+    <xacro:property name="THRUSTER_Y" value="0.09"/>
+    <xacro:property name="THRUSTER_Z" value="-0.009"/>
+    <xacro:property name="VERT_THRUSTER_Y" value="0.105"/>
+    <xacro:property name="VERT_THRUSTER_Z" value="0.09"/>
+    <xacro:property name="MASS_Z" value="0.011"/>
+    <xacro:property name="FORWARD_FORCE" value="50"/>
+    <xacro:property name="REVERSE_FORCE" value="40"/>
+    <xacro:property name="HAS_TETHER" default="false"/>
+    <xacro:property name="SURFACE" default="0"/>
+    <!-- Physics properties -->
+    <xacro:property name="FLUID_DENSITY" value="997"/>
+    <xacro:property name="DISPLACED_MASS" value="${TOTAL_VOLUME*FLUID_DENSITY}"/>
+    <!-- General constants -->
+    <xacro:property name="PI" value="3.1415926535897931"/>
+    <!-- Materials -->
+    <material name="gray">
+        <color rgba="0.5 0.5 0.5 1.0"/>
+    </material>
+    <material name="blue">
+        <color rgba="0.5 0.5 1.0 1.0"/>
+    </material>
+    <material name="red">
+        <color rgba="1.0 0.0 0.0 1.0"/>
+    </material>
+    <!-- Thruster origins -->
+    <xacro:property name="front_right_origin">
+        <origin xyz="${THRUSTER_X} ${-THRUSTER_Y} ${THRUSTER_Z}" rpy="0 ${PI/2} ${PI/4}"/>
+    </xacro:property>
+    <xacro:property name="front_left_origin">
+        <origin xyz="${THRUSTER_X} ${THRUSTER_Y} ${THRUSTER_Z}" rpy="0 ${PI/2} ${-PI/4}"/>
+    </xacro:property>
+    <xacro:property name="rear_right_origin">
+        <origin xyz="${-THRUSTER_X} ${-THRUSTER_Y} ${THRUSTER_Z}" rpy="0 ${PI/2} ${PI*3/4}"/>
+    </xacro:property>
+    <xacro:property name="rear_left_origin">
+        <origin xyz="${-THRUSTER_X} ${THRUSTER_Y} ${THRUSTER_Z}" rpy="0 ${PI/2} ${-PI*3/4}"/>
+    </xacro:property>
+    <xacro:property name="vertical_right_origin">
+        <origin xyz="0 ${-VERT_THRUSTER_Y} ${VERT_THRUSTER_Z}" rpy="0 0 0"/>
+    </xacro:property>
+    <xacro:property name="vertical_left_origin">
+        <origin xyz="0 ${VERT_THRUSTER_Y} ${VERT_THRUSTER_Z}" rpy="0 0 0"/>
+    </xacro:property>
+    <!-- Thruster macro -->
+    <xacro:macro name="t200" params="name *origin">
+        <link name="t200_link_${name}">
+            <!-- Front cone -->
+            <visual>
+                <origin xyz="0 0 0"/>
+                <geometry>
+                    <sphere radius="0.02"/>
+                </geometry>
+                <material name="gray"/> <!-- All visual elements in this link pick up this material -->
+            </visual>
+            <!-- Rear cone -->
+            <visual>
+                <origin xyz="0 0 -0.07"/>
+                <geometry>
+                    <sphere radius="0.02"/>
+                </geometry>
+            </visual>
+            <!-- Thruster body -->
+            <visual>
+                <origin xyz="0 0 -0.035"/>
+                <geometry>
+                    <cylinder length="0.07" radius="0.02"/>
+                </geometry>
+            </visual>
+            <!-- Propeller guard -->
+            <visual>
+                <origin xyz="0 0 -0.0225"/>
+                <geometry>
+                    <cylinder length="0.045" radius="0.045"/>
+                </geometry>
+            </visual>
+        </link>
+        <joint name="t200_joint_${name}" type="fixed">
+            <xacro:insert_block name="origin"/>
+            <parent link="base_link"/>
+            <child link="t200_link_${name}"/>
+        </joint>
+    </xacro:macro>
+    <!-- Base link -->
+    <link name="base_link">
+        <!-- Inertial -->
+        <inertial>
+            <origin xyz="0 0 ${MASS_Z}"/> <!-- Center of mass -->
+            <mass value="${TOTAL_MASS}"/>
+            <inertia ixx="${IXX}" ixy="0.0" ixz="0.0" iyy="${IYY}" iyz="0.0" izz="${IZZ}"/>
+        </inertial>
+        <!-- Float -->
+        <visual>
+            <origin xyz="${FLOAT_X} ${FLOAT_Y} ${FLOAT_Z}"/>
+            <geometry>
+                <box size="0.15 0.09 0.08"/>
+            </geometry>
+            <material name="blue"/>
+        </visual>
+        <!-- Float -->
+        <visual>
+            <origin xyz="${FLOAT_X} ${-FLOAT_Y} ${FLOAT_Z}"/>
+            <geometry>
+                <box size="0.15 0.09 0.08"/>
+            </geometry>
+        </visual>
+        <!-- Float -->
+        <visual>
+            <origin xyz="${-FLOAT_X} ${FLOAT_Y} ${FLOAT_Z}"/>
+            <geometry>
+                <box size="0.15 0.09 0.08"/>
+            </geometry>
+        </visual>
+        <!-- Float -->
+        <visual>
+            <origin xyz="${-FLOAT_X} ${-FLOAT_Y} ${FLOAT_Z}"/>
+            <geometry>
+                <box size="0.15 0.09 0.08"/>
+            </geometry>
+        </visual>
+        <!-- Electronics tube -->
+        <visual>
+            <origin xyz="0 0 0.063" rpy="0 ${PI/2} 0"/>
+            <geometry>
+                <cylinder length="0.32" radius="0.055"/>
+            </geometry>
+        </visual>
+        <!-- Battery tube -->
+        <visual>
+            <origin xyz="0 0 -0.05" rpy="0 ${PI/2} 0"/>
+            <geometry>
+                <cylinder length="0.25" radius="0.045"/>
+            </geometry>
+        </visual>
+        <!-- Left down-facing camera tube -->
+        <visual>
+            <origin xyz="-0.15 0.18 0" rpy="0 0 0"/>
+            <geometry>
+                <cylinder length="0.135" radius="0.0275"/>
+            </geometry>
+        </visual>
+        <!-- Right down-facing camera tube -->
+        <visual>
+            <origin xyz="-0.15 -0.18 0" rpy="0 0 0"/>
+            <geometry>
+                <cylinder length="0.135" radius="0.0275"/>
+            </geometry>
+        </visual>
+        <!-- Collision region -->
+        <collision>
+            <geometry>
+                <box size="${LENGTH} ${WIDTH} ${HEIGHT}"/>
+            </geometry>
+        </collision>
     </link>
-    <joint name="t200_joint_${name}" type="fixed">
-      <xacro:insert_block name="origin" />
-      <parent link="base_link"/>
-      <child link="t200_link_${name}"/>
-    </joint>
-  </xacro:macro>
-  <!-- Base link -->
-  <link name="base_link">
-    <!-- Inertial -->
-    <inertial>
-      <origin xyz="0 0 ${MASS_Z}"/> <!-- Center of mass -->
-      <mass value="${TOTAL_MASS}"/>
-      <inertia ixx="${IXX}" ixy="0.0" ixz="0.0" iyy="${IYY}" iyz="0.0" izz="${IZZ}"/>
-    </inertial>
-    <!-- Float -->
-    <visual>
-      <origin xyz="${FLOAT_X} ${FLOAT_Y} ${FLOAT_Z}"/>
-      <geometry><box size="0.15 0.09 0.08"/></geometry>
-      <material name="blue"/>
-    </visual>
-    <!-- Float -->
-    <visual>
-      <origin xyz="${FLOAT_X} ${-FLOAT_Y} ${FLOAT_Z}"/>
-      <geometry><box size="0.15 0.09 0.08"/></geometry>
-    </visual>
-    <!-- Float -->
-    <visual>
-      <origin xyz="${-FLOAT_X} ${FLOAT_Y} ${FLOAT_Z}"/>
-      <geometry><box size="0.15 0.09 0.08"/></geometry>
-    </visual>
-    <!-- Float -->
-    <visual>
-      <origin xyz="${-FLOAT_X} ${-FLOAT_Y} ${FLOAT_Z}"/>
-      <geometry><box size="0.15 0.09 0.08"/></geometry>
-    </visual>
-    <!-- Electronics tube -->
-    <visual>
-      <origin xyz="0 0 0.063" rpy="0 ${PI/2} 0"/>
-      <geometry><cylinder length="0.32" radius="0.055"/></geometry>
-    </visual>
-    <!-- Front-facing camera hemisphere -->
-    <visual>
-      <origin xyz="0.16 0 0.063" rpy="0 ${PI/2} 0"/>
-      <geometry><sphere radius="0.052"/></geometry>
-    </visual>
-    <!-- Battery tube -->
-    <visual>
-      <origin xyz="0 0 -0.05" rpy="0 ${PI/2} 0"/>
-      <geometry><cylinder length="0.25" radius="0.045"/></geometry>
-    </visual>
-    <!-- Left down-facing camera tube -->
-    <visual>
-      <origin xyz="-0.15 0.18 0" rpy="0 0 0"/>
-      <geometry><cylinder length="0.135" radius="0.0275"/></geometry>
-    </visual>
-    <!-- Right down-facing camera tube -->
-    <visual>
-      <origin xyz="-0.15 -0.18 0" rpy="0 0 0"/>
-      <geometry><cylinder length="0.135" radius="0.0275"/></geometry>
-    </visual>
-    <!-- Collision region -->
-    <collision>
-      <geometry><box size="${LENGTH} ${WIDTH} ${HEIGHT}"/></geometry>
-    </collision>
-  </link>
-  <!-- Left down-facing camera -->
-  <link name="left_camera_link">
-    <!-- Camera hemisphere -->
-    <visual>
-      <origin xyz="0 0 0" rpy="0 0 0"/>
-      <geometry><sphere radius="0.026"/></geometry>
-      <material name="red"/>
-    </visual>
-  </link>
-  <!-- Attach left down-facing camera to base_link -->
-  <joint name="left_camera_joint" type="fixed">
-    <axis xyz="0 1 0" />
-    <origin xyz="-0.15 0.18 -0.0675" rpy="0 ${PI/2} 0"/>
-    <parent link="base_link"/>
-    <child link="left_camera_link"/>
-  </joint>
-  <!-- Right down-facing camera -->
-  <link name="right_camera_link">
-    <!-- Camera hemisphere -->
-    <visual>
-      <origin xyz="0 0 0" rpy="0 0 0"/>
-      <geometry><sphere radius="0.026"/></geometry>
-      <material name="red"/>
-    </visual>
-  </link>
-  <!-- Attach right down-facing camera to base_link -->
-  <joint name="right_camera_joint" type="fixed">
-    <axis xyz="0 1 0" />
-    <origin xyz="-0.15 -0.18 -0.0675" rpy="0 1.57079 0"/>
-    <parent link="base_link"/>
-    <child link="right_camera_link"/>
-  </joint>
-  <!-- Attach thrusters to the base_link -->
-  <xacro:t200 name="front_right">
-    <xacro:insert_block name="front_right_origin"/>
-  </xacro:t200>
-  <xacro:t200 name="front_left">
-    <xacro:insert_block name="front_left_origin"/>
-  </xacro:t200>
-  <xacro:t200 name="rear_right">
-    <xacro:insert_block name="rear_right_origin"/>
-  </xacro:t200>
-  <xacro:t200 name="rear_left">
-    <xacro:insert_block name="rear_left_origin"/>
-  </xacro:t200>
-  <xacro:t200 name="vertical_right">
-    <xacro:insert_block name="vertical_right_origin"/>
-  </xacro:t200>
-  <xacro:t200 name="vertical_left">
-    <xacro:insert_block name="vertical_left_origin"/>
-  </xacro:t200>
-  <!--
-    The OrcaBuoyancyPlugin applies a force that counteracts gravity.
-    Buoyancy force is not applied if the link is above the surface of the water.
+    <!-- Barometer link TODO /tf too low -->
+    <link name="baro_link">
+        <visual>
+            <origin xyz="0 0 0.05" rpy="0 ${PI/2} 0"/>
+            <geometry>
+                <cylinder length="0.01" radius="0.01"/>
+            </geometry>
+            <material name="red"/>
+        </visual>
+    </link>
+    <!-- Attach baro_link to base_link -->
+    <joint name="baro_joint" type="fixed">
+        <origin xyz="-0.16 0 0" rpy="0 0 0"/>
+        <parent link="base_link"/>
+        <child link="baro_link"/>
+    </joint>
+    <!-- Forward camera link -->
+    <link name="forward_camera_link">
+        <visual>
+            <origin xyz="0 0 0" rpy="0 0 0"/>
+            <geometry>
+                <sphere radius="0.052"/>
+            </geometry>
+            <material name="red"/>
+        </visual>
+    </link>
+    <!-- Attach forward_camera_link to base_link -->
+    <joint name="forward_camera_joint" type="fixed">
+        <origin xyz="0.16 0 0.063" rpy="0 0 0"/>
+        <parent link="base_link"/>
+        <child link="forward_camera_link"/>
+    </joint>
+    <!-- Forward camera frame -->
+    <link name="forward_camera_frame"/>
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