Commit message: Add 2nd camera, flip to portrait, can now run 9m between markers in simulation

File: orca_description/urdf/orca.urdf (robot description, URDF)
Before this commit: robot orca, 14 links, 13 joints
Links:
- link left_camera_link: geometry visual box size=0.01 0.04 0.03
- link right_camera_link: geometry visual box size=0.01 0.04 0.03
Joints:
- joint forward_camera_frame_joint: origin xyz=0.16 0 0.063 rpy=-1.57079632679 0 -1.57079632679 -> xyz=0.16 0 0.063 rpy=-1.5707963267948966 0 -1.5707963267948966
- joint left_camera_frame_joint: origin xyz=-0.15 0.18 -0.0675 rpy=3.14159265359 0 -1.57079632679 -> xyz=-0.15 0.18 -0.0675 rpy=0 3.141592653589793 0
- joint left_camera_joint: axis 0 1 0 -> (none); origin xyz=-0.15 0.18 -0.0675 rpy=0 1.57079632679 0 -> xyz=-0.15 0.18 -0.0675 rpy=1.5707963267948966 1.5707963267948966 0
- joint right_camera_frame_joint: origin xyz=-0.15 -0.18 -0.0675 rpy=3.14159265359 0 -1.57079632679 -> xyz=-0.15 -0.18 -0.0675 rpy=0 3.141592653589793 0
- joint right_camera_joint: axis 0 1 0 -> (none); origin xyz=-0.15 -0.18 -0.0675 rpy=0 1.57079 0 -> xyz=-0.15 -0.18 -0.0675 rpy=1.5707963267948966 1.5707963267948966 0
- joint t200_joint_front_left: origin xyz=0.15 0.09 -0.009 rpy=0 1.57079632679 -0.785398163397 -> xyz=0.15 0.09 -0.009 rpy=0 1.5707963267948966 -0.7853981633974483
- joint t200_joint_front_right: origin xyz=0.15 -0.09 -0.009 rpy=0 1.57079632679 0.785398163397 -> xyz=0.15 -0.09 -0.009 rpy=0 1.5707963267948966 0.7853981633974483
- joint t200_joint_rear_left: origin xyz=-0.15 0.09 -0.009 rpy=0 1.57079632679 -2.35619449019 -> xyz=-0.15 0.09 -0.009 rpy=0 1.5707963267948966 -2.356194490192345
- joint t200_joint_rear_right: origin xyz=-0.15 -0.09 -0.009 rpy=0 1.57079632679 2.35619449019 -> xyz=-0.15 -0.09 -0.009 rpy=0 1.5707963267948966 2.356194490192345

File: orca_description/urdf/orca.urdf.xacro (robot description, xacro)
@@ -208,4 +208,5 @@
         <child link="forward_camera_frame"/>
     </joint>
+    <!-- Left and right cameras are positioned to see markers along the seafloor. Both are portrait. -->
     <!-- Left camera link -->
     <link name="left_camera_link">
@@ -213,5 +214,6 @@
             <origin xyz="0 0 0" rpy="0 0 0"/>
             <geometry>
-                <sphere radius="0.026"/>
+                <!-- Make the aspect ratio obvious -->
+                <box size="0.01 0.04 0.03"/>
             </geometry>
             <material name="red"/>
@@ -220,6 +222,5 @@
     <!-- Attach left_camera_link to base_link -->
     <joint name="left_camera_joint" type="fixed">
-        <axis xyz="0 1 0"/>
-        <origin xyz="-0.15 0.18 -0.0675" rpy="0 ${PI/2} 0"/>
+        <origin xyz="-0.15 0.18 -0.0675" rpy="${PI/2} ${PI/2} 0"/>
         <parent link="base_link"/>
         <child link="left_camera_link"/>
@@ -229,5 +230,5 @@
     <!-- Attach left_camera_frame to base_link (parsed by filter_node)  -->
     <joint name="left_camera_frame_joint" type="fixed">
-        <origin xyz="-0.15 0.18 -0.0675" rpy="${PI} 0 ${-PI/2}"/>
+        <origin xyz="-0.15 0.18 -0.0675" rpy="0 ${PI} 0"/>
         <parent link="base_link"/>
         <child link="left_camera_frame"/>
@@ -235,9 +236,9 @@
     <!-- Right camera link -->
     <link name="right_camera_link">
-        <!-- Camera hemisphere -->
         <visual>
             <origin xyz="0 0 0" rpy="0 0 0"/>
             <geometry>
-                <sphere radius="0.026"/>
+                <!-- Make the aspect ratio obvious -->
+                <box size="0.01 0.04 0.03"/>
             </geometry>
             <material name="red"/>
@@ -246,6 +247,5 @@
     <!-- Attach right_camera_link to base_link -->
     <joint name="right_camera_joint" type="fixed">
-        <axis xyz="0 1 0"/>
-        <origin xyz="-0.15 -0.18 -0.0675" rpy="0 1.57079 0"/>
+        <origin xyz="-0.15 -0.18 -0.0675" rpy="${PI/2} ${PI/2} 0"/>
         <parent link="base_link"/>
         <child link="right_camera_link"/>
@@ -253,7 +253,7 @@
     <!-- Right camera frame -->
     <link name="right_camera_frame"/>
-    <!-- Attach right_camera_frame to base_link -->
+    <!-- Attach right_camera_frame to base_link (parsed by filter_node) -->
     <joint name="right_camera_frame_joint" type="fixed">
-        <origin xyz="-0.15 -0.18 -0.0675" rpy="${PI} 0 ${-PI/2}"/>
+        <origin xyz="-0.15 -0.18 -0.0675" rpy="0 ${PI} 0"/>
         <parent link="base_link"/>
         <child link="right_camera_frame"/>
@@ -312,6 +312,5 @@
         <plugin name="OrcaThrusterPlugin" filename="libOrcaThrusterPlugin.so">
             <link_name>orca::base_link</link_name>
-            <thruster
-                    name="front_right"> <!-- name attributes are ignored; the tag order must match the message array order -->
+            <thruster name="front_right"> <!-- name attributes are ignored; the tag order must match the message array order -->
                 <pos_force>${FORWARD_FORCE}</pos_force> <!-- units are N, positive for ccw, negative for cw -->
                 <neg_force>${REVERSE_FORCE}</neg_force> <!-- units are N, positive for ccw, negative for cw -->
@@ -371,13 +370,13 @@
     This xacro macro attaches a camera to ${prefix}_camera_link:
   -->
-    <xacro:macro name="camera_plugin" params="prefix">
+    <xacro:macro name="camera_plugin" params="prefix width height horizontal_fov">
         <gazebo reference="${prefix}_camera_link">
             <sensor type="camera" name="${prefix}_camera">
                 <update_rate>30.0</update_rate>
                 <camera name="head">
-                    <horizontal_fov>1.4</horizontal_fov>
+                    <horizontal_fov>${horizontal_fov}</horizontal_fov>
                     <image>
-                        <width>800</width>
-                        <height>600</height>
+                        <width>${width}</width>
+                        <height>${height}</height>
                         <format>R8G8B8</format>
                     </image>
@@ -415,7 +414,7 @@
 <!--    <xacro:camera_plugin prefix="forward"/>-->
     <!-- Left down-facing camera: -->
-    <xacro:camera_plugin prefix="left"/>
+    <xacro:camera_plugin prefix="left" width="800" height="600" horizontal_fov="1.4"/>
     <!-- Right down-facing camera: -->
-<!--    <xacro:camera_plugin prefix="right"/>-->
+    <xacro:camera_plugin prefix="right" width="800" height="600" horizontal_fov="1.4"/>
     <gazebo>
         <plugin name="p3d_test" filename="libgazebo_ros_p3d.so">
