Commit message: CMake Builds maps and worlds, remove tether drag, comment drag a bit better

File: orca_description/xacro/orca.urdf.xacro (robot description, xacro)
@@ -1,5 +1,11 @@
 <?xml version="1.0"?>
 <robot name="orca" xmlns:xacro="http://ros.org/wiki/xacro">
-    <!-- Orca constants -->
+    <!--
+        Orca constants
+        Flight dynamics are hugely driven by these 3 constants, all in the body frame:
+            {x, y, THRUSTER_Z}: where forward/back/strafe/yaw thrust forces are applied
+            {0, 0, MASS_Z}: where the linear and angular drag force is applied
+            {0, 0, VOLUME_Z}: where the buoyancy force is applied
+     -->
     <xacro:property name="TOTAL_MASS" value="9.75"/>  <!-- 9.75 floats in freshwater, 10.0 for seawater -->
     <xacro:property name="TOTAL_VOLUME" value="0.01"/>
@@ -19,4 +25,5 @@
     <xacro:property name="VERT_THRUSTER_Z" value="0.09"/>
     <xacro:property name="MASS_Z" value="0.011"/>
+    <xacro:property name="VOLUME_Z" value="0.06"/>
     <xacro:property name="FORWARD_FORCE" value="50"/>
     <xacro:property name="REVERSE_FORCE" value="40"/>
@@ -286,5 +293,5 @@
             <fluid_density>${FLUID_DENSITY}</fluid_density>
             <link name="base_link">
-                <center_of_volume>0 0 0.06</center_of_volume>
+                <center_of_volume>0 0 ${VOLUME_Z}</center_of_volume>
                 <volume>${TOTAL_VOLUME}</volume>
             </link>
@@ -298,4 +305,5 @@
             <link name="base_link">
                 <center_of_mass>0 0 ${MASS_Z}</center_of_mass>
+                <center_of_volume>0 0 ${VOLUME_Z}</center_of_volume>
                 <tether_attach>-0.25 0 ${THRUSTER_Z}</tether_attach>
                 <xacro:unless value="${HAS_TETHER}">

Commit message: Fixed z problems, increased bollard z force from 40 to 44, etc.

File: orca_description/xacro/orca.urdf.xacro (robot description, xacro)
@@ -12,5 +12,5 @@
     <xacro:property name="LENGTH" value="0.457"/>
     <xacro:property name="WIDTH" value="0.338"/>
-    <xacro:property name="HEIGHT" value="0.254"/>
+    <xacro:property name="HEIGHT" value="0.25"/>
     <xacro:property name="IXX" value="${TOTAL_MASS / 12 * (WIDTH * WIDTH + HEIGHT * HEIGHT)}"/>
     <xacro:property name="IYY" value="${TOTAL_MASS / 12 * (LENGTH * LENGTH + HEIGHT * HEIGHT)}"/>
@@ -27,5 +27,5 @@
     <xacro:property name="VOLUME_Z" value="0.06"/>
     <xacro:property name="FORWARD_FORCE" value="50"/>
-    <xacro:property name="REVERSE_FORCE" value="40"/>
+    <xacro:property name="REVERSE_FORCE" value="44"/>
     <xacro:property name="HAS_TETHER" default="false"/>
     <xacro:property name="SURFACE" default="0"/>
@@ -175,8 +175,8 @@
         </collision>
     </link>
-    <!-- Barometer link TODO /tf too low -->
+    <!-- Barometer link -->
     <link name="baro_link">
         <visual>
-            <origin xyz="0 0 0.05" rpy="0 ${PI/2} 0"/>
+            <origin xyz="0 0 0" rpy="0 ${PI/2} 0"/>
             <geometry>
                 <cylinder length="0.01" radius="0.01"/>
@@ -187,5 +187,5 @@
     <!-- Attach baro_link to base_link -->
     <joint name="baro_joint" type="fixed">
-        <origin xyz="-0.16 0 0" rpy="0 0 0"/>
+        <origin xyz="-0.16 0 0.05" rpy="0 0 0"/>
         <parent link="base_link"/>
         <child link="baro_link"/>

Commit message: Split vertical bollard force into up and down

File: orca_description/xacro/orca.urdf.xacro (robot description, xacro)
@@ -27,5 +27,5 @@
     <xacro:property name="VOLUME_Z" value="0.06"/>
     <xacro:property name="FORWARD_FORCE" value="50"/>
-    <xacro:property name="REVERSE_FORCE" value="44"/>
+    <xacro:property name="REVERSE_FORCE" value="40"/>
     <xacro:property name="HAS_TETHER" default="false"/>
     <xacro:property name="SURFACE" default="0"/>

Commit message: Add drag experiments, can be used to calc drag in the field

File: orca_description/xacro/orca.urdf.xacro (robot description, xacro)
@@ -7,6 +7,11 @@
             {0, 0, MASS_Z}: where the linear and angular drag force is applied
             {0, 0, VOLUME_Z}: where the buoyancy force is applied
+        Default simulation is fresh water and slightly positive buoyancy:
+            TOTAL_VOLUME = 0.01
+            FLUID_DENSITY = 997
+            DISPLACED_MASS = TOTAL_VOLUME * FLUID_DENSITY = 9.97
+            TOTAL_MASS = 9.9
      -->
-    <xacro:property name="TOTAL_MASS" value="9.75"/>  <!-- 9.75 floats in freshwater, 10.0 for seawater -->
+    <xacro:property name="TOTAL_MASS" value="9.9"/>
     <xacro:property name="TOTAL_VOLUME" value="0.01"/>
     <xacro:property name="LENGTH" value="0.457"/>
@@ -32,5 +37,4 @@
     <!-- Physics properties -->
     <xacro:property name="FLUID_DENSITY" value="997"/>
-    <xacro:property name="DISPLACED_MASS" value="${TOTAL_VOLUME*FLUID_DENSITY}"/>
     <!-- General constants -->
     <xacro:property name="PI" value="3.1415926535897931"/>

Commit message: Fix small bugs while tuning 'hold pressure'

File: orca_description/xacro/orca.urdf.xacro (robot description, xacro)
@@ -37,4 +37,6 @@
     <!-- Physics properties -->
     <xacro:property name="FLUID_DENSITY" value="997"/>
+    <!-- Sensor properties, should match orca_shared/model.hpp -->
+    <xacro:property name="BARO_FREQ" value="23.0"/>
     <!-- General constants -->
     <xacro:property name="PI" value="3.1415926535897931"/>
@@ -358,5 +360,5 @@
     <gazebo reference="baro_link">
         <sensor name="barometer_sensor" type="altimeter">
-            <update_rate>24</update_rate> <!-- Match measured barometer_node rate -->
+            <update_rate>${BARO_FREQ}</update_rate>
             <plugin name="OrcaBarometerPlugin" filename="libOrcaBarometerPlugin.so">
                 <fluid_density>${FLUID_DENSITY}</fluid_density>

Commit message: Work on pose_filter and PID tuning in simulation

File: orca_description/xacro/orca.urdf.xacro (robot description, xacro)
@@ -39,4 +39,5 @@
     <!-- Sensor properties, should match orca_shared/model.hpp -->
     <xacro:property name="BARO_FREQ" value="23.0"/>
+    <xacro:property name="CAMERA_FREQ" value="30.0"/>
     <!-- General constants -->
     <xacro:property name="PI" value="3.1415926535897931"/>
@@ -384,5 +385,5 @@
         <gazebo reference="${prefix}_camera_link">
             <sensor type="camera" name="${prefix}_camera">
-                <update_rate>30.0</update_rate>
+                <update_rate>${CAMERA_FREQ}</update_rate>
                 <camera name="head">
                     <horizontal_fov>${horizontal_fov}</horizontal_fov>
